File: navelino.sch (KiCad schematic (older format))
At the start: 70 parts, among them IC1 ATMEGA328P-A, P1 CONN_5X2, P3 CONN_6, SW0 SW_PUSH, SW1 SW_PUSH, SW2 SW_PUSH, U1 CJA1117B-3.3, X0 CRYSTAL

Commit message: Actualizado el regulador a algo más pequeño :)
Parts:
- removed C1: 10uF, Capacitors_Tantalum_SMD:TantalC_SizeA_EIA-3216_HandSoldering, symbol CPsmall
- removed C2: 22uF, Capacitors_Tantalum_SMD:TantalC_SizeB_EIA-3528_HandSoldering, symbol CPsmall
- added C1: 0.1uF, Capacitors_SMD:C_0603, symbol Csmall
- added C2: 1uF, Capacitors_SMD:C_0603, symbol Csmall
- U1: value CJA1117B-3.3 -> XC6204B332MR; footprint Housings_SOT-89:SOT89-3_Housing_Handsoldering -> Housings_SOT-23_SOT-143_TSOT-6:SOT-23-5; symbol NCP1117ST33T3G -> LD3985G122R; SEEED 1310120P1 -> 310030046
Connections:
- no-connect marks 0 -> 1
Changed lines of the file:
@@
 LIBS:contrib
 LIBS:valves
-LIBS:notenom-cache
+LIBS:navelino-cache
 EELAYER 25 0
 EELAYER END
@@
 RESET
 $Comp
-L NCP1117ST33T3G U1
+L LD3985G122R U1
 U 1 1 558CA477
 P 3750 1200
 F 0 "U1" H 3900 1004 40  0000 C CNN
-F 1 "CJA1117B-3.3" H 3750 1400 40  0000 C CNN
-F 2 "Housings_SOT-89:SOT89-3_Housing_Handsoldering" H 3750 1200 60  0001 C CNN
+F 1 "XC6204B332MR" H 3750 1400 40  0000 C CNN
+F 2 "Housings_SOT-23_SOT-143_TSOT-6:SOT-23-5" H 3750 1200 60  0001 C CNN
 F 3 "" H 3750 1200 60  0000 C CNN
-F 4 "1310120P1" H 3750 1200 60  0001 C CNN "SEEED"
+F 4 "310030046" H 3750 1200 60  0001 C CNN "SEEED"
 	1    3750 1200
 	1    0    0    -1
 $EndComp
-$Comp
-L CPsmall C1
-U 1 1 558D4895
-P 3100 1250
-F 0 "C1" H 3125 1300 30  0000 L CNN
-F 1 "10uF" H 3125 1175 30  0000 L CNN
-F 2 "Capacitors_Tantalum_SMD:TantalC_SizeA_EIA-3216_HandSoldering" H 3100 1250 60  0001 C CNN
-F 3 "" H 3100 1250 60  0000 C CNN
-F 4 "302020002" H 3100 1250 60  0001 C CNN "SEEED"
-	1    3100 1250
-	1    0    0    -1
-$EndComp
-$Comp
-L CPsmall C2
-U 1 1 558D48E1
-P 4400 1250
-F 0 "C2" H 4425 1300 30  0000 L CNN
-F 1 "22uF" H 4425 1175 30  0000 L CNN
-F 2 "Capacitors_Tantalum_SMD:TantalC_SizeB_EIA-3528_HandSoldering" H 4400 1250 60  0001 C CNN
-F 3 "" H 4400 1250 60  0000 C CNN
-F 4 "302020021" H 4400 1250 60  0001 C CNN "SEEED"
-	1    4400 1250
-	1    0    0    -1
-$EndComp
-Wire Wire Line
-	3100 1350 3100 1450
-Wire Wire Line
-	3100 1450 4400 1450
-Wire Wire Line
-	4400 1450 4400 1350
-Connection ~ 3750 1450
-Wire Wire Line
-	2800 1150 3350 1150
-Wire Wire Line
-	4150 1150 4400 1150
+Wire Wire Line
+	2800 1150 3300 1150
 Text GLabel 2800 1150 0    39   Input ~ 0
 RAW
@@
 $EndComp
 Wire Wire Line
-	4400 1150 4400 1100
+	4400 1100 4400 1300
 $Comp
 L GND #PWR08
 U 1 1 558D4E13
-P 3750 1550
-F 0 "#PWR08" H 3750 1550 30  0001 C CNN
-F 1 "GND" H 3750 1480 30  0001 C CNN
-F 2 "" H 3750 1550 60  0000 C CNN
-F 3 "" H 3750 1550 60  0000 C CNN
-	1    3750 1550
-	1    0    0    -1
-$EndComp
-Wire Wire Line
-	3750 1550 3750 1450
+P 3750 1600
+F 0 "#PWR08" H 3750 1600 30  0001 C CNN
+F 1 "GND" H 3750 1530 30  0001 C CNN
+F 2 "" H 3750 1600 60  0000 C CNN
+F 3 "" H 3750 1600 60  0000 C CNN
+	1    3750 1600
+	1    0    0    -1
+$EndComp
 $Comp
 L CONN_6 P3
@@
 L PWR_FLAG #FLG010
 U 1 1 558ED2B2
-P 3100 1450
-F 0 "#FLG010" H 3100 1545 30  0001 C CNN
-F 1 "PWR_FLAG" H 3100 1630 30  0000 C CNN
-F 2 "" H 3100 1450 60  0000 C CNN
-F 3 "" H 3100 1450 60  0000 C CNN
-	1    3100 1450
+P 3100 1500
+F 0 "#FLG010" H 3100 1595 30  0001 C CNN
+F 1 "PWR_FLAG" H 3100 1680 30  0000 C CNN
+F 2 "" H 3100 1500 60  0000 C CNN
+F 3 "" H 3100 1500 60  0000 C CNN
+	1    3100 1500
 	-1   0    0    1
 $EndComp
@@
 Wire Wire Line
 	1600 4500 1900 4500
+$Comp
+L Csmall C1
+U 1 1 559028A0
+P 3100 1400
+F 0 "C1" H 3125 1450 30  0000 L CNN
+F 1 "0.1uF" H 3125 1350 30  0000 L CNN
+F 2 "Capacitors_SMD:C_0603" H 3100 1400 60  0001 C CNN
+F 3 "" H 3100 1400 60  0000 C CNN
+F 4 "302010138" H 3100 1400 60  0001 C CNN "SEEED"
+	1    3100 1400
+	1    0    0    -1
+$EndComp
+$Comp
+L Csmall C2
+U 1 1 55902AFC
+P 4400 1400
+F 0 "C2" H 4425 1450 30  0000 L CNN
+F 1 "1uF" H 4425 1350 30  0000 L CNN
+F 2 "Capacitors_SMD:C_0603" H 4400 1400 60  0001 C CNN
+F 3 "" H 4400 1400 60  0000 C CNN
+F 4 "302010139" H 4400 1400 60  0001 C CNN "SEEED"
+	1    4400 1400
+	1    0    0    -1
+$EndComp
+NoConn ~ 4200 1300
+Wire Wire Line
+	4200 1150 4400 1150
+Wire Wire Line
+	3100 1300 3100 1150
+Wire Wire Line
+	3100 1300 3300 1300
+Wire Wire Line
+	3100 1500 4400 1500
+Connection ~ 4400 1150
+Connection ~ 3750 1500
+Wire Wire Line
+	3750 1500 3750 1600
 $EndSCHEMATC

Commit message: Cambiados casi todos los componentes de 06 a 08 para que pueda funcionar como taller de soldadura SMD Añadido el Jumper para poder desactivar los leds y usar los pines libremente
Parts:
- D1, D2, D3: footprint LEDs:LED-0603 -> LEDs:LED-0805; SEEED 304090045 -> 304090061
- D10, D4, D5, D6, D7, D8, D9: footprint LEDs:LED-0603 -> LEDs:LED-0805
- JP1, JP10, JP2, JP3, JP4, JP5, JP6, JP7, JP8, JP9: footprint (none) -> tmw:PCB_JUMPER
- R1, R2, R3: footprint Resistors_SMD:R_0603_HandSoldering -> Resistors_SMD:R_0805_HandSoldering; SEEED 301010300 -> 301010364
- R10, R4, R5, R6, R7, R8, R9: footprint Resistors_SMD:R_0603_HandSoldering -> Resistors_SMD:R_0805_HandSoldering
Changed lines of the file:
@@
 F 0 "D1" H 7500 2450 50  0000 C CNN
 F 1 "BLUE" H 7500 2250 50  0000 C CNN
-F 2 "LEDs:LED-0603" H 7500 2350 60  0001 C CNN
+F 2 "LEDs:LED-0805" H 7500 2350 60  0001 C CNN
 F 3 "" H 7500 2350 60  0000 C CNN
-F 4 "304090045" H 7500 2350 60  0001 C CNN "SEEED"
+F 4 "304090061" H 7500 2350 60  0001 C CNN "SEEED"
 	1    7500 2350
 	1    0    0    -1
@@
 F 0 "D2" H 7500 2750 50  0000 C CNN
 F 1 "BLUE" H 7500 2550 50  0000 C CNN
-F 2 "LEDs:LED-0603" H 7500 2650 60  0001 C CNN
+F 2 "LEDs:LED-0805" H 7500 2650 60  0001 C CNN
 F 3 "" H 7500 2650 60  0000 C CNN
-F 4 "304090045" H 7500 2650 60  0001 C CNN "SEEED"
+F 4 "304090061" H 7500 2650 60  0001 C CNN "SEEED"
 	1    7500 2650
 	1    0    0    -1
@@
 F 0 "D3" H 7500 3050 50  0000 C CNN
 F 1 "BLUE" H 7500 2850 50  0000 C CNN
-F 2 "LEDs:LED-0603" H 7500 2950 60  0001 C CNN
+F 2 "LEDs:LED-0805" H 7500 2950 60  0001 C CNN
 F 3 "" H 7500 2950 60  0000 C CNN
-F 4 "304090045" H 7500 2950 60  0001 C CNN "SEEED"
+F 4 "304090061" H 7500 2950 60  0001 C CNN "SEEED"
 	1    7500 2950
 	1    0    0    -1
@@
 F 0 "D4" H 7500 3350 50  0000 C CNN
 F 1 "LED" H 7500 3150 50  0000 C CNN
-F 2 "LEDs:LED-0603" H 7500 3250 60  0001 C CNN
+F 2 "LEDs:LED-0805" H 7500 3250 60  0001 C CNN
 F 3 "" H 7500 3250 60  0000 C CNN
 	1    7500 3250
@@
 F 0 "D5" H 7500 3650 50  0000 C CNN
 F 1 "LED" H 7500 3450 50  0000 C CNN
-F 2 "LEDs:LED-0603" H 7500 3550 60  0001 C CNN
+F 2 "LEDs:LED-0805" H 7500 3550 60  0001 C CNN
 F 3 "" H 7500 3550 60  0000 C CNN
 	1    7500 3550
@@
 F 0 "D6" H 7500 3950 50  0000 C CNN
 F 1 "LED" H 7500 3750 50  0000 C CNN
-F 2 "LEDs:LED-0603" H 7500 3850 60  0001 C CNN
+F 2 "LEDs:LED-0805" H 7500 3850 60  0001 C CNN
 F 3 "" H 7500 3850 60  0000 C CNN
 	1    7500 3850
@@
 F 0 "D7" H 7500 4250 50  0000 C CNN
 F 1 "LED" H 7500 4050 50  0000 C CNN
-F 2 "LEDs:LED-0603" H 7500 4150 60  0001 C CNN
+F 2 "LEDs:LED-0805" H 7500 4150 60  0001 C CNN
 F 3 "" H 7500 4150 60  0000 C CNN
 	1    7500 4150
@@
 F 0 "D8" H 7500 4550 50  0000 C CNN
 F 1 "LED" H 7500 4350 50  0000 C CNN
-F 2 "LEDs:LED-0603" H 7500 4450 60  0001 C CNN
+F 2 "LEDs:LED-0805" H 7500 4450 60  0001 C CNN
 F 3 "" H 7500 4450 60  0000 C CNN
 	1    7500 4450
@@
 F 0 "R1" V 7130 2350 40  0000 C CNN
 F 1 "330" V 7057 2351 40  0000 C CNN
-F 2 "Resistors_SMD:R_0603_HandSoldering" V 6980 2350 30  0001 C CNN
+F 2 "Resistors_SMD:R_0805_HandSoldering" V 6980 2350 30  0001 C CNN
 F 3 "" H 7050 2350 30  0000 C CNN
-F 4 "301010300" V 7050 2350 60  0001 C CNN "SEEED"
+F 4 "301010364" V 7050 2350 60  0001 C CNN "SEEED"
 	1    7050 2350
 	0    -1   -1   0
@@
 F 0 "R2" V 7130 2650 40  0000 C CNN
 F 1 "330" V 7057 2651 40  0000 C CNN
-F 2 "Resistors_SMD:R_0603_HandSoldering" V 6980 2650 30  0001 C CNN
+F 2 "Resistors_SMD:R_0805_HandSoldering" V 6980 2650 30  0001 C CNN
 F 3 "" H 7050 2650 30  0000 C CNN
-F 4 "301010300" V 7050 2650 60  0001 C CNN "SEEED"
+F 4 "301010364" V 7050 2650 60  0001 C CNN "SEEED"
 	1    7050 2650
 	0    -1   -1   0
@@
 F 0 "R3" V 7130 2950 40  0000 C CNN
 F 1 "330" V 7057 2951 40  0000 C CNN
-F 2 "Resistors_SMD:R_0603_HandSoldering" V 6980 2950 30  0001 C CNN
+F 2 "Resistors_SMD:R_0805_HandSoldering" V 6980 2950 30  0001 C CNN
 F 3 "" H 7050 2950 30  0000 C CNN
-F 4 "301010300" V 7050 2950 60  0001 C CNN "SEEED"
+F 4 "301010364" V 7050 2950 60  0001 C CNN "SEEED"
 	1    7050 2950
 	0    -1   -1   0
@@
 F 0 "R4" V 7130 3250 40  0000 C CNN
 F 1 "330" V 7057 3251 40  0000 C CNN
-F 2 "Resistors_SMD:R_0603_HandSoldering" V 6980 3250 30  0001 C CNN
+F 2 "Resistors_SMD:R_0805_HandSoldering" V 6980 3250 30  0001 C CNN
 F 3 "" H 7050 3250 30  0000 C CNN
 F 4 "301010300" V 7050 3250 60  0001 C CNN "SEEED"
@@
 F 0 "R5" V 7130 3550 40  0000 C CNN
 F 1 "330" V 7057 3551 40  0000 C CNN
-F 2 "Resistors_SMD:R_0603_HandSoldering" V 6980 3550 30  0001 C CNN
+F 2 "Resistors_SMD:R_0805_HandSoldering" V 6980 3550 30  0001 C CNN
 F 3 "" H 7050 3550 30  0000 C CNN
 F 4 "301010300" V 7050 3550 60  0001 C CNN "SEEED"
@@
 F 0 "R6" V 7130 3850 40  0000 C CNN
 F 1 "330" V 7057 3851 40  0000 C CNN
-F 2 "Resistors_SMD:R_0603_HandSoldering" V 6980 3850 30  0001 C CNN
+F 2 "Resistors_SMD:R_0805_HandSoldering" V 6980 3850 30  0001 C CNN
 F 3 "" H 7050 3850 30  0000 C CNN
 F 4 "301010300" V 7050 3850 60  0001 C CNN "SEEED"
@@
 F 0 "R7" V 7130 4150 40  0000 C CNN
 F 1 "330" V 7057 4151 40  0000 C CNN
-F 2 "Resistors_SMD:R_0603_HandSoldering" V 6980 4150 30  0001 C CNN
+F 2 "Resistors_SMD:R_0805_HandSoldering" V 6980 4150 30  0001 C CNN
 F 3 "" H 7050 4150 30  0000 C CNN
 F 4 "301010300" V 7050 4150 60  0001 C CNN "SEEED"
@@
 F 0 "R8" V 7130 4450 40  0000 C CNN
 F 1 "330" V 7057 4451 40  0000 C CNN
-F 2 "Resistors_SMD:R_0603_HandSoldering" V 6980 4450 30  0001 C CNN
+F 2 "Resistors_SMD:R_0805_HandSoldering" V 6980 4450 30  0001 C CNN
 F 3 "" H 7050 4450 30  0000 C CNN
 F 4 "301010300" V 7050 4450 60  0001 C CNN "SEEED"
@@
 F 0 "D9" H 7500 4800 50  0000 C CNN
 F 1 "LED" H 7500 4600 50  0000 C CNN
-F 2 "LEDs:LED-0603" H 7500 4700 60  0001 C CNN
+F 2 "LEDs:LED-0805" H 7500 4700 60  0001 C CNN
 F 3 "" H 7500 4700 60  0000 C CNN
 	1    7500 4700
@@
 F 0 "D10" H 7500 5100 50  0000 C CNN
 F 1 "LED" H 7500 4900 50  0000 C CNN
-F 2 "LEDs:LED-0603" H 7500 5000 60  0001 C CNN
+F 2 "LEDs:LED-0805" H 7500 5000 60  0001 C CNN
 F 3 "" H 7500 5000 60  0000 C CNN
 	1    7500 5000
@@
 F 0 "R9" V 7130 4700 40  0000 C CNN
 F 1 "330" V 7057 4701 40  0000 C CNN
-F 2 "Resistors_SMD:R_0603_HandSoldering" V 6980 4700 30  0001 C CNN
+F 2 "Resistors_SMD:R_0805_HandSoldering" V 6980 4700 30  0001 C CNN
 F 3 "" H 7050 4700 30  0000 C CNN
 F 4 "301010300" V 7050 4700 60  0001 C CNN "SEEED"
@@
 F 0 "R10" V 7130 5000 40  0000 C CNN
 F 1 "330" V 7057 5001 40  0000 C CNN
-F 2 "Resistors_SMD:R_0603_HandSoldering" V 6980 5000 30  0001 C CNN
+F 2 "Resistors_SMD:R_0805_HandSoldering" V 6980 5000 30  0001 C CNN
 F 3 "" H 7050 5000 30  0000 C CNN
 F 4 "301010300" V 7050 5000 60  0001 C CNN "SEEED"
@@
 F 0 "JP1" H 6500 2500 60  0000 C CNN
 F 1 "JUMPER" H 6500 2270 40  0000 C CNN
-F 2 "" H 6500 2350 60  0001 C CNN
+F 2 "tmw:PCB_JUMPER" H 6500 2350 60  0001 C CNN
 F 3 "" H 6500 2350 60  0000 C CNN
 	1    6500 2350
@@
 F 0 "JP2" H 6500 2800 60  0000 C CNN
 F 1 "JUMPER" H 6500 2570 40  0000 C CNN
-F 2 "" H 6500 2650 60  0001 C CNN
+F 2 "tmw:PCB_JUMPER" H 6500 2650 60  0001 C CNN
 F 3 "" H 6500 2650 60  0000 C CNN
 	1    6500 2650
@@
 F 0 "JP3" H 6500 3100 60  0000 C CNN
 F 1 "JUMPER" H 6500 2870 40  0000 C CNN
-F 2 "" H 6500 2950 60  0001 C CNN
+F 2 "tmw:PCB_JUMPER" H 6500 2950 60  0001 C CNN
 F 3 "" H 6500 2950 60  0000 C CNN
 	1    6500 2950
@@
 F 0 "JP4" H 6500 3400 60  0000 C CNN
 F 1 "JUMPER" H 6500 3170 40  0000 C CNN
-F 2 "" H 6500 3250 60  0001 C CNN
+F 2 "tmw:PCB_JUMPER" H 6500 3250 60  0001 C CNN
 F 3 "" H 6500 3250 60  0000 C CNN
 	1    6500 3250
@@
 F 0 "JP5" H 6500 3700 60  0000 C CNN
 F 1 "JUMPER" H 6500 3470 40  0000 C CNN
-F 2 "" H 6500 3550 60  0001 C CNN
+F 2 "tmw:PCB_JUMPER" H 6500 3550 60  0001 C CNN
 F 3 "" H 6500 3550 60  0000 C CNN
 	1    6500 3550
@@
 F 0 "JP6" H 6500 4000 60  0000 C CNN
 F 1 "JUMPER" H 6500 3770 40  0000 C CNN
-F 2 "" H 6500 3850 60  0001 C CNN
+F 2 "tmw:PCB_JUMPER" H 6500 3850 60  0001 C CNN
 F 3 "" H 6500 3850 60  0000 C CNN
 	1    6500 3850
@@
 F 0 "JP7" H 6500 4300 60  0000 C CNN
 F 1 "JUMPER" H 6500 4070 40  0000 C CNN
-F 2 "" H 6500 4150 60  0001 C CNN
+F 2 "tmw:PCB_JUMPER" H 6500 4150 60  0001 C CNN
 F 3 "" H 6500 4150 60  0000 C CNN
 	1    6500 4150
@@
 F 0 "JP8" H 6500 4600 60  0000 C CNN
 F 1 "JUMPER" H 6500 4370 40  0000 C CNN
-F 2 "" H 6500 4450 60  0001 C CNN
+F 2 "tmw:PCB_JUMPER" H 6500 4450 60  0001 C CNN
 F 3 "" H 6500 4450 60  0000 C CNN
 	1    6500 4450
@@
 F 0 "JP9" H 6500 4850 60  0000 C CNN
 F 1 "JUMPER" H 6500 4620 40  0000 C CNN
-F 2 "" H 6500 4700 60  0001 C CNN
+F 2 "tmw:PCB_JUMPER" H 6500 4700 60  0001 C CNN
 F 3 "" H 6500 4700 60  0000 C CNN
 	1    6500 4700
@@
 F 0 "JP10" H 6500 5150 60  0000 C CNN
 F 1 "JUMPER" H 6500 4920 40  0000 C CNN
-F 2 "" H 6500 5000 60  0001 C CNN
+F 2 "tmw:PCB_JUMPER" H 6500 5000 60  0001 C CNN
 F 3 "" H 6500 5000 60  0000 C CNN
 	1    6500 5000

Commit message: Finalizado el routing!
Parts:
- removed SW1, SW2: SW_PUSH, Buttons_Switches_SMD:SW_SPST_PTS645, symbol SW_PUSH
- added CON1: USB-MINI-B, SEEED:ST-USB-001G, symbol USB-MINI-B
- added SW1, SW2: SMD-SWITCH-TACTILE-SPST-NO(4P-D6.0MM), SEEED:SW4-SMD-6.0X6.0X5.0MM, symbol SMD-SWITCH-TACTILE-SPST-NO(4P-D6.0MM)
- C1: footprint Capacitors_SMD:C_0603 -> Capacitors_SMD:C_0805; SEEED 302010138 -> 302010165
- C2: footprint Capacitors_SMD:C_0603 -> Capacitors_SMD:C_0805; SEEED 302010139 -> 302010179
- C3, C4, C7: footprint Capacitors_SMD:C_0603_HandSoldering -> Capacitors_SMD:C_0805; SEEED 302010138 -> 302010165
- C5, C6: footprint Capacitors_SMD:C_0603_HandSoldering -> Capacitors_SMD:C_0805; SEEED 302010143 -> 302010151
- D10, D4, D5, D6, D7, D8, D9: SEEED (none) -> 304090046
- IC1: SEEED (none) -> 310010049
- JP1, JP10, JP2, JP3, JP4, JP5, JP6, JP7, JP8, JP9: footprint tmw:PCB_JUMPER -> Wire_Connections_Bridges:PCB_JUMPER
- P1: footprint (none) -> SEEED:df12(3.0)-10ds-0.5v
- R0: footprint Resistors_SMD:R_0603_HandSoldering -> Resistors_SMD:R_0805_HandSoldering; SEEED 301010299 -> 301010361
- SW0: footprint (none) -> SEEED:B3U-1000P; SEEED (none) -> 311020047
- U1: footprint Housings_SOT-23_SOT-143_TSOT-6:SOT-23-5 -> TO_SOT_Packages_SMD:SOT-23-5
- X0: footprint (none) -> SMD-CRYSTAL-8MHZ-20PF-20PPM_2P-5.0X3.2MM_:X2-SMD-5.0X3.2X1.3MM
Connections:
- net PB3 is gone; now on net PB3/MOSI: JP3.1, PB3.1
- net PB4 is gone; now on net PB4/MISO: JP4.1, PB4.1
- net SCK/PB5 is gone; now on net PB5/SCK: JP5.1, PB5.1
- net DTR: no longer P1.7
- net GND: now also P1.6, CON1.5 (GND), SW1.3 (B1), SW2.3 (B1); no longer P1.10, P1.9
- net PB0: now also SW2.1 (A0)
- net PB1: now also JP6.1; no longer JP1.1
- net PB2: now also JP7.1; no longer JP2.1
- net PB3/MOSI: now also P1.4; no longer P1.6
- net PB4/MISO: now also P1.1; no longer P1.4
- net PB5/SCK: now also P1.3; no longer P1.8
- net PC0: no longer JP6.1
- net PC1: no longer JP7.1
- net PC2: now also SW1.1 (A0); no longer JP8.1
- net PD2: now also JP1.1
- net PD3: now also JP2.1
- net PD5: now also JP8.1
- net RAW: now also CON1.1 (VBUS)
- net RESET: now also P1.5; no longer P1.2
- net RXI: no longer P1.5
- net TXO: no longer P1.3
- net VCC: now also P1.2; no longer P1.1
- no-connect marks 1 -> 16
Other:
- moved on the sheet: C4, P3, R0, SW0

Commit message: Un poco de amor para el Silkscreen
Parts:
- removed CON1: USB-MINI-B, SEEED:ST-USB-001G, symbol USB-MINI-B
- added CON1: USB, SEEED:ST-USB-001G, symbol CONN_5
- C5, C6: value 22pF -> 27pF; SEEED 302010151 -> 302010150
- X0: SEEED 306010004 -> 306010047
Connections:
- net GND: now also CON1.5
- net RAW: now also CON1.1
- no-connect marks 16 -> 12
Changed lines of the file:
@@
 F 2 "SMD-CRYSTAL-8MHZ-20PF-20PPM_2P-5.0X3.2MM_:X2-SMD-5.0X3.2X1.3MM" H 5200 1350 60  0001 C CNN
 F 3 "" H 5200 1350 60  0000 C CNN
-F 4 "306010004" H 5200 1350 60  0001 C CNN "SEEED"
+F 4 "306010047" H 5200 1350 60  0001 C CNN "SEEED"
 	1    5200 1350
 	0    1    1    0
@@
 $EndComp
 Wire Wire Line
-	3050 4350 3050 4750
+	3050 4350 3050 4450
+Wire Wire Line
+	3050 4450 3050 4550
+Wire Wire Line
+	3050 4550 3050 4750
 Connection ~ 3050 4550
 Connection ~ 3050 4450
 Wire Wire Line
-	3050 2150 3050 2550
+	3050 2150 3050 2250
+Wire Wire Line
+	3050 2250 3050 2350
+Wire Wire Line
+	3050 2350 3050 2550
 Connection ~ 3050 2350
 Wire Wire Line
@@
 Connection ~ 3050 2250
 Wire Wire Line
-	7700 2050 7700 5550
+	7700 2050 7700 2350
+Wire Wire Line
+	7700 2350 7700 2650
+Wire Wire Line
+	7700 2650 7700 2950
+Wire Wire Line
+	7700 2950 7700 3250
+Wire Wire Line
+	7700 3250 7700 3550
+Wire Wire Line
+	7700 3550 7700 3850
+Wire Wire Line
+	7700 3850 7700 4150
+Wire Wire Line
+	7700 4150 7700 4450
+Wire Wire Line
+	7700 4450 7700 4700
+Wire Wire Line
+	7700 4700 7700 5000
+Wire Wire Line
+	7700 5000 7700 5500
+Wire Wire Line
+	7700 5500 7700 5550
 Connection ~ 7700 4150
 Connection ~ 7700 3850
@@
 $EndComp
 Wire Wire Line
-	2800 1150 3300 1150
+	2800 1150 3100 1150
+Wire Wire Line
+	3100 1150 3300 1150
 Text GLabel 2800 1150 0    39   Input ~ 0
 RAW
@@
 $EndComp
 Wire Wire Line
-	4400 1100 4400 1300
+	4400 1100 4400 1150
+Wire Wire Line
+	4400 1150 4400 1300
 $Comp
 L GND #PWR08
@@
 P 5400 1050
 F 0 "C5" H 5400 1150 40  0000 L CNN
-F 1 "22pF" H 5406 965 40  0000 L CNN
+F 1 "27pF" H 5406 965 40  0000 L CNN
 F 2 "Capacitors_SMD:C_0805" H 5438 900 30  0001 C CNN
 F 3 "" H 5400 1050 60  0000 C CNN
-F 4 "302010151" H 5400 1050 60  0001 C CNN "SEEED"
+F 4 "302010150" H 5400 1050 60  0001 C CNN "SEEED"
 	1    5400 1050
 	0    1    1    0
@@
 P 5400 1650
 F 0 "C6" H 5400 1750 40  0000 L CNN
-F 1 "22pF" H 5406 1565 40  0000 L CNN
+F 1 "27pF" H 5406 1565 40  0000 L CNN
 F 2 "Capacitors_SMD:C_0805" H 5438 1500 30  0001 C CNN
 F 3 "" H 5400 1650 60  0000 C CNN
-F 4 "302010151" H 5400 1650 60  0001 C CNN "SEEED"
+F 4 "302010150" H 5400 1650 60  0001 C CNN "SEEED"
 	1    5400 1650
 	0    1    1    0
 $EndComp
 Wire Wire Line
-	5600 1050 5600 1650
+	5600 1050 5600 1350
+Wire Wire Line
+	5600 1350 5600 1650
 $Comp
 L GND #PWR011
@@
 	2900 2850 3050 2850
 Wire Wire Line
-	1650 5000 1950 5000
+	1650 5000 1800 5000
+Wire Wire Line
+	1800 5000 1950 5000
 $Comp
 L Csmall C1
@@
 	3100 1300 3300 1300
 Wire Wire Line
-	3100 1500 4400 1500
+	3100 1500 3750 1500
+Wire Wire Line
+	3750 1500 4400 1500
 Connection ~ 4400 1150
 Connection ~ 3750 1500
 Wire Wire Line
 	3750 1500 3750 1600
-$Comp
-L USB-MINI-B CON1
-U 1 1 566BF372
-P 4000 5600
-F 0 "CON1" H 3750 6050 60  0000 C CNN
-F 1 "USB-MINI-B" H 3950 5100 60  0000 C CNN
-F 2 "SEEED:ST-USB-001G" H 4000 5600 60  0001 C CNN
-F 3 "" H 4000 5600 60  0000 C CNN
-F 4 "320010000" H 4000 5600 60  0001 C CNN "SEEED"
-	1    4000 5600
-	1    0    0    -1
-$EndComp
-Text GLabel 3450 5900 0    39   Input ~ 0
+Text GLabel 1050 4200 0    39   Input ~ 0
 GND
-Text GLabel 3450 5300 0    39   Input ~ 0
+Text GLabel 1050 3800 0    39   Input ~ 0
 RAW
-NoConn ~ 4550 5900
-NoConn ~ 4550 5750
-NoConn ~ 4550 5450
-NoConn ~ 4550 5300
-NoConn ~ 3450 5750
-NoConn ~ 3450 5600
-NoConn ~ 3450 5450
 $Comp
 L CONN_5X2 P1
@@
 Connection ~ 7700 5500
 NoConn ~ 7500 5300
+$Comp
+L CONN_5 CON1
+U 1 1 56704FE0
+P 1450 4000
+F 0 "CON1" V 1400 4000 50  0000 C CNN
+F 1 "USB" V 1500 4000 50  0000 C CNN
+F 2 "SEEED:ST-USB-001G" H 1450 4000 60  0001 C CNN
+F 3 "" H 1450 4000 60  0000 C CNN
+	1    1450 4000
+	1    0    0    -1
+$EndComp
+NoConn ~ 1050 3900
+NoConn ~ 1050 4000
+NoConn ~ 1050 4100
 $EndSCHEMATC

Commit message: Condensadores de X0 cambiados a 27pF Añadidos orificios de montaje de 3mm
Parts:
- added M1, M2: CONN_1, Wire_Pads:SolderWirePad_single_1mmDrill, symbol CONN_1
Connections:
- no-connect marks 12 -> 14
Changed lines of the file:
@@
 $EndComp
 Wire Wire Line
-	3050 4350 3050 4450
-Wire Wire Line
-	3050 4450 3050 4550
-Wire Wire Line
-	3050 4550 3050 4750
+	3050 4350 3050 4750
 Connection ~ 3050 4550
 Connection ~ 3050 4450
 Wire Wire Line
-	3050 2150 3050 2250
-Wire Wire Line
-	3050 2250 3050 2350
-Wire Wire Line
-	3050 2350 3050 2550
+	3050 2150 3050 2550
 Connection ~ 3050 2350
 Wire Wire Line
@@
 Connection ~ 3050 2250
 Wire Wire Line
-	7700 2050 7700 2350
-Wire Wire Line
-	7700 2350 7700 2650
-Wire Wire Line
-	7700 2650 7700 2950
-Wire Wire Line
-	7700 2950 7700 3250
-Wire Wire Line
-	7700 3250 7700 3550
-Wire Wire Line
-	7700 3550 7700 3850
-Wire Wire Line
-	7700 3850 7700 4150
-Wire Wire Line
-	7700 4150 7700 4450
-Wire Wire Line
-	7700 4450 7700 4700
-Wire Wire Line
-	7700 4700 7700 5000
-Wire Wire Line
-	7700 5000 7700 5500
-Wire Wire Line
-	7700 5500 7700 5550
+	7700 2050 7700 5550
 Connection ~ 7700 4150
 Connection ~ 7700 3850
@@
 $EndComp
 Wire Wire Line
-	2800 1150 3100 1150
-Wire Wire Line
-	3100 1150 3300 1150
+	2800 1150 3300 1150
 Text GLabel 2800 1150 0    39   Input ~ 0
 RAW
@@
 $EndComp
 Wire Wire Line
-	4400 1100 4400 1150
-Wire Wire Line
-	4400 1150 4400 1300
+	4400 1100 4400 1300
 $Comp
 L GND #PWR08
@@
 $EndComp
 Wire Wire Line
-	5600 1050 5600 1350
-Wire Wire Line
-	5600 1350 5600 1650
+	5600 1050 5600 1650
 $Comp
 L GND #PWR011
@@
 	2900 2850 3050 2850
 Wire Wire Line
-	1650 5000 1800 5000
-Wire Wire Line
-	1800 5000 1950 5000
+	1650 5000 1950 5000
 $Comp
 L Csmall C1
@@
 	3100 1300 3300 1300
 Wire Wire Line
-	3100 1500 3750 1500
-Wire Wire Line
-	3750 1500 4400 1500
+	3100 1500 4400 1500
 Connection ~ 4400 1150
 Connection ~ 3750 1500
@@
 NoConn ~ 1050 4000
 NoConn ~ 1050 4100
+$Comp
+L CONN_1 M1
+U 1 1 567431FA
+P 6550 700
+F 0 "M1" H 6630 700 40  0000 L CNN
+F 1 "CONN_1" H 6550 755 30  0001 C CNN
+F 2 "Wire_Pads:SolderWirePad_single_1mmDrill" H 6550 700 60  0001 C CNN
+F 3 "" H 6550 700 60  0000 C CNN
+	1    6550 700
+	1    0    0    -1
+$EndComp
+$Comp
+L CONN_1 M2
+U 1 1 567432F1
+P 6550 850
+F 0 "M2" H 6630 850 40  0000 L CNN
+F 1 "CONN_1" H 6550 905 30  0001 C CNN
+F 2 "Wire_Pads:SolderWirePad_single_1mmDrill" H 6550 850 60  0001 C CNN
+F 3 "" H 6550 850 60  0000 C CNN
+	1    6550 850
+	1    0    0    -1
+$EndComp
+NoConn ~ 6400 700
+NoConn ~ 6400 850
 $EndSCHEMATC
