File: navelino.sch (KiCad schematic (older format))
At the start: 73 parts, among them CON1 USB, IC1 ATMEGA328P-A, M1 CONN_1, M2 CONN_1, P1 CONN_5X2, P3 CONN_6, SW0 SW_PUSH, SW1 SMD-SWITCH-TACTILE-SPST-NO(4P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, SW2 SMD-SWITCH-TACTILE-SPST-NO(4P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, U1 XC6204B332MR, X0 CRYSTAL

Commit message: Empezando a meter las dependencias de librerías dentro del proyecto Substituido el conector de la hoja por algo más standard
Parts:
- removed P1: CONN_5X2, SEEED:df12(3.0)-10ds-0.5v, symbol CONN_5X2
- added P1: CONN_02X03, navelino:ISPSMD, symbol CONN_02X03
- ADC6, ADC7, M1, M2, PB0, PB1, PB2, PB3, PB4, PB5, PC0, PC1, PC2, PC3, PC4, PC5, PC6, PD2, PD3, PD4, PD5, PD6, PD7, PGND1, PRAW1, PVCC1: footprint Wire_Pads:SolderWirePad_single_1mmDrill -> navelino:SolderWirePad_single_1mmDrill
- C1, C2: footprint Capacitors_SMD:C_0805 -> navelino:C_0805
- C3, C4, C5, C6, C7: footprint Capacitors_SMD:C_0805 -> navelino:C_0805; symbol C -> C-RESCUE-navelino
- CON1: footprint SEEED:ST-USB-001G -> navelino:ST-USB-001G
- D1, D10, D2, D3, D4, D5, D6, D7, D8, D9: footprint LEDs:LED-0805 -> navelino:LED-0805; symbol LED -> LED-RESCUE-navelino
- IC1: footprint Housings_QFP:TQFP-32_7x7mm_Pitch0.8mm -> navelino:TQFP-32_7x7mm_Pitch0.8mm; symbol ATMEGA328P-A -> ATMEGA328P-A-RESCUE-navelino
- JP1, JP10, JP2, JP3, JP4, JP5, JP6, JP7, JP8, JP9: footprint Wire_Connections_Bridges:PCB_JUMPER -> navelino:PCB_JUMPER
- P3: footprint Pin_Headers:Pin_Header_Angled_1x06 -> navelino:Pin_Header_Angled_1x06
- R0, R1, R10, R2, R3, R4, R5, R6, R7, R8, R9: footprint Resistors_SMD:R_0805_HandSoldering -> navelino:R_0805_HandSoldering; symbol R -> R-RESCUE-navelino
- SW0: footprint SEEED:B3U-1000P -> navelino:B3U-1000P
- SW1, SW2: footprint SEEED:SW4-SMD-6.0X6.0X5.0MM -> navelino:SW4-SMD-6.0X6.0X5.0MM
- U1: footprint TO_SOT_Packages_SMD:SOT-23-5 -> navelino:SOT-23-5
- X0: footprint SMD-CRYSTAL-8MHZ-20PF-20PPM_2P-5.0X3.2MM_:X2-SMD-5.0X3.2X1.3MM -> navelino:X2-SMD-5.0X3.2X1.3MM
Connections:
- no-connect marks 14 -> 10
